File: hardware/shoes/rev_a/shoes.sch (EAGLE design)
At the start: 45 parts, among them J4 TC2030-JLINK-NL, Q1 MOSFET-NCHANNELXFDN-3, Q2 MOSFET-NCHANNELXFDN-3, Q3 MOSFET-NCHANNELXFDN-3, Q4 MOSFET-NCHANNELXFDN-3, U1 NRF51822QF, U2 ADXL362, X1 16MHz

Commit message: new PCB preliminary working
Connections:
- removed net P25: U1.P25
Changed lines of the file:
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@@
-</segment>
-</net>
-<net name="P25" class="0">
-<segment>
-<pinref part="U1" gate="G$1" pin="P25"/>
-<wire x1="160.02" y1="101.6" x2="162.56" y2="101.6" width="0.1524" layer="91"/>
 </segment>
 </net>
